File: hardware/pcb/variable_brightness_led_lamp/LED_Lamp_v1.kicad_pcb (KiCad board)
At the start: 2 copper layers, 130 x 130 mm, 25 parts, among them J1 54-00166, Q1 2N3904, SW1 RotaryEncoder_Switch

Commit message: firmware-update, PCB-final
Parts:
- moved M2 13.7 mm to (117.1, 119.0)
- moved M2 13.2 mm to (182.9, 119.0)
- moved M2 10.0 mm to (150.0, 62.0)
- renumbered REF** to M2
Routing:
- net /5V: track 252.8 -> 259.8 mm
- net /B_Rot_Enc: track 91.0 -> 94.3 mm
